Commit message: Port TETRA DS4-M to ROS 2 Humble and include navigation build files

File: tetra_description/urdf/base.urdf.xacro (robot description, xacro)
@@ -1,10 +1,12 @@
 <?xml version="1.0"?>
-<robot name="tetra" xmlns:xacro="http://www.ros.org/wiki/xacro">
+<robot name="tetra" xmlns:xacro="http://ros.org/wiki/xacro">
   <!-- Define a number of dimensions using properties -->
-  <xacro:property name="base_length" value="0.6127" />
-  <xacro:property name="base_radius" value="0.2452" />
+  <xacro:property name="base_length" value="0.473" />
+  <xacro:property name="base_radius" value="0.2365" />
+  <xacro:property name="wheel_length" value="0.047" />
+  <xacro:property name="wheel_radius" value="0.085" />
   <xacro:property name="wheel_offset_x" value="0.0" />
-  <xacro:property name="wheel_offset_y" value="0.220" />
-  <xacro:property name="wheel_offset_z" value="-0.1005" />
+  <xacro:property name="wheel_offset_y" value="0.207" /> <!--0.220-->
+  <xacro:property name="wheel_offset_z" value="-0.100" />
   <xacro:property name="PI" value="3.1415926" />
   <xacro:macro name="cylinder_inertia" params="m r h">
@@ -22,7 +24,7 @@
     <origin xyz=" 0 ${-1.0*wheel_offset_y} 0 " rpy="0 0 0" />
 	<geometry>
-	  <mesh filename="package://tetra_description/meshes/wheel_drive_left.stl" scale="0.001 0.001 0.001" />
+	  <mesh filename="package://tetra_description/meshes/ds4_m/wheel_drive_left.stl" scale="0.001 0.001 0.001" />
 	</geometry>
-	<material name="darkgrey"/>
+	<material name="DarkGrey"/>
   </visual>
     </link>
@@ -37,18 +39,19 @@
     <origin xyz=" 0 ${wheel_offset_y} 0 " rpy="0 0 0" />
 	<geometry>
-	  <mesh filename="package://tetra_description/meshes/wheel_drive_right.stl" scale="0.001 0.001 0.001" />
+	  <mesh filename="package://tetra_description/meshes/ds4_m/wheel_drive_right.stl" scale="0.001 0.001 0.001" />
 	</geometry>
-	<material name="darkgrey"/>
+	<material name="DarkGrey"/>
   </visual>
     </link>
   <!-- The base xacro macro -->
-   <link name= "base_link">
+  <xacro:macro name="base" params="name color">
+   <link name="${name}_link">
     <visual>
     <origin xyz=" 0 0 0 " rpy="0 0 0" />
       <geometry>
         <mesh
-          filename="package://tetra_description/meshes/platform_body.stl" scale="0.001 0.001 0.001" />
+          filename="package://tetra_description/meshes/ds4_m/platform_body_lower.stl" scale="0.001 0.001 0.001" />
       </geometry>
-      <material name="black"/>
+      <material name="Black"/>
     </visual>
       <collision>
@@ -59,11 +62,12 @@
       </collision>
     </link>
+  </xacro:macro>
   <link name="base_footprint">
       <visual>
-        <origin xyz="-0.08935 0 0" rpy="0 0 0" />
+        <origin xyz="-0.125 0 0" rpy="0 0 0" />
         <geometry>
-	  <box size="0.6127 0.4904 0.001" />
+	  <box size="0.730 0.520 0.001" />
         </geometry>
-        <material name="transparentgreen" />
+        <material name="TransparentGreen" />
       </visual>
   </link>
@@ -74,16 +78,17 @@
   </joint>
   <!-- Rear Caster-->
-   <link name="rear_caster_rotate">
+  <xacro:macro name="rear_caster_wheel" params="prefix dir">
+        <link name="${prefix}_rear_caster_rotate">
             <visual>
                 <origin xyz="0 0 0" rpy="0 0 0"/>
                 <geometry>
-                    <mesh filename="package://tetra_description/meshes/caster_yoke.stl" scale="0.001 0.001 0.001" />
+                    <mesh filename="package://tetra_description/meshes/ds4_m/caster_yoke.stl" scale="0.001 0.001 0.001" />
                 </geometry>
-                <material name="darkgrey" />
+                <material name="DarkGrey" />
             </visual>
             <collision>
                 <origin xyz="0 0 0" rpy="0 0 0"/>
                 <geometry>
-                    <mesh filename="package://tetra_description/meshes/caster_yoke.stl" scale="0.001 0.001 0.001" />
+                    <mesh filename="package://tetra_description/meshes/ds4_m/caster_yoke.stl" scale="0.001 0.001 0.001" />
                 </geometry>
             </collision>
@@ -94,22 +99,22 @@
             </inertial>
         </link>
-        <joint name="rear_caster_rotate_joint" type="fixed">
+        <joint name="${prefix}_rear_caster_rotate_joint" type="fixed">
             <parent link="base_link"/>
-            <child link="rear_caster_rotate"/>
-            <origin xyz="-0.300 0 0" rpy="0 0 0"/>
+            <child link="${prefix}_rear_caster_rotate"/>
+            <origin xyz="-0.300 ${dir*-0.160} -0.0225" rpy="0 0 0"/>
             <axis xyz="0 0 1"/>
         </joint>
-        <link name="rear_caster_wheel">
+        <link name="${prefix}_rear_caster_wheel">
             <visual>
                 <origin xyz="0 0 0" rpy="0 0 0"/>
                 <geometry>
-                    <mesh filename="package://tetra_description/meshes/caster_wheel.stl" scale="0.001 0.001 0.001" />
+                    <mesh filename="package://tetra_description/meshes/ds4_m/caster_wheel.stl" scale="0.001 0.001 0.001" />
                 </geometry>
-                <material name="darkgrey" />
+                <material name="DarkGrey" />
             </visual>
             <collision>
                 <origin xyz="0 0 0" rpy="0 0 0"/>
                 <geometry>
-                    <mesh filename="package://tetra_description/meshes/caster_wheel.stl" scale="0.001 0.001 0.001" />
+                    <mesh filename="package://tetra_description/meshes/ds4_m/caster_wheel.stl" scale="0.001 0.001 0.001" />
                 </geometry>
             </collision>
@@ -120,9 +125,12 @@
             </inertial>
         </link>
-        <joint name="rear_caster_wheel_joint" type="fixed">
-            <parent link="rear_caster_rotate"/>
-            <child link="rear_caster_wheel"/>
-            <origin xyz="-0.03 0 -0.06291" rpy="0 0 0"/>
+        <joint name="${prefix}_rear_caster_wheel_joint" type="fixed">
+            <parent link="${prefix}_rear_caster_rotate"/>
+            <child link="${prefix}_rear_caster_wheel"/>
+            <origin xyz="-0.022 0 -0.047" rpy="0 0 0"/>
             <axis xyz="0 1 0"/>
         </joint>
+    </xacro:macro>
+  <xacro:rear_caster_wheel prefix="l" dir="1"/>
+  <xacro:rear_caster_wheel prefix="r" dir="-1"/>
 </robot>

File: tetra_description/urdf/materials.urdf.xacro (robot description, xacro)
@@ -2,44 +2,44 @@
 <robot>
   <!-- Put all the color definitions in a separate file -->
-  <material name="black">
+  <material name="Black">
     <color rgba="0.2 0.2 0.2 1.0"/>
   </material>
-   <material name="transparentblack">
+   <material name="TransparentBlack">
     <color rgba="0.2 0.2 0.2 1.0"/>
   </material>
-  <material name="orange">
+  <material name="Orange">
     <color rgba="1.0  0.55 0.0 1.0"/>
   </material>
-  <material name="grey">
+  <material name="Grey">
     <color rgba="0.7 0.7 0.7 1.0"/>
   </material>
-  <material name="darkgrey">
+  <material name="DarkGrey">
     <color rgba="0.4 0.4 0.4 1.0"/>
   </material>
-  <material name="red">
+  <material name="Red">
     <color rgba="0.8 0.0 0.0 1.0"/>
   </material>
-  <material name="transparentred">
+  <material name="TransparentRed">
     <color rgba="0.5 0.1 0.1 1.0"/>
   </material>
-  <material name="white">
+  <material name="White">
     <color rgba="1.0 1.0 1.0 0.98"/>
   </material>
-  <material name="offWhite">
+  <material name="OffWhite">
     <color rgba="0.8 0.8 0.8 1.0"/>
   </material>
-  <material name="blue">
+  <material name="Blue">
     <color rgba="0.0 0.0 0.8 1.0"/>
   </material>
-  <material name="green">
+  <material name="Green">
     <color rgba="0.0 0.8 0.0 1.0"/>
   </material>
-  <material name="transparentgreen">
+  <material name="TransparentGreen">
     <color rgba="0.0 0.8 0.0 0.5"/>
   </material>
- <material name="transparentblue">
+ <material name="TransparentBlue">
     <color rgba="0.0 0.0 0.6 0.8"/>
   </material>
- <material name="transparentyellow">
+ <material name="TransparentYellow">
     <color rgba="0.8 0.8 0.1 1.0"/>
   </material>

File: tetra_description/urdf/tetra.xacro (robot description, xacro)
@@ -1,4 +1,11 @@
 <?xml version="1.0"?>
 <robot name="tetra" xmlns:xacro="http://www.ros.org/wiki/xacro">
+  <!-- Mount defaults match the directly received DS4-M tetra_description.xacro. -->
+  <xacro:arg name="lidar_x" default="0.1372"/>
+  <xacro:arg name="lidar_y" default="0.0"/>
+  <xacro:arg name="lidar_z" default="0.142"/>
+  <xacro:arg name="lidar_roll" default="3.14"/>
+  <xacro:arg name="lidar_pitch" default="3.14"/>
+  <xacro:arg name="lidar_yaw" default="0.0"/>
   <!-- Define a number of dimensions using properties -->
   <xacro:property name="base_length" value="0.473" />
@@ -17,5 +24,5 @@
    <xacro:include filename="$(find tetra_description)/urdf/base.urdf.xacro" />
    <!-- Add the base and wheels -->
-   <base name="base" color="black"/>
+   <xacro:base name="base" color="Black"/>
   <link name="laser">
       <visual>
@@ -24,9 +31,10 @@
           <box size="0.01 0.01 0.01" />
         </geometry>
-        <material name="grey" />
+        <material name="Grey" />
       </visual>
   </link>
   <joint name="base_link_to_laser_link" type="fixed">
-    <origin xyz="0.1372 0 0.142" rpy="0 0 0" />
+    <origin xyz="$(arg lidar_x) $(arg lidar_y) $(arg lidar_z)"
+            rpy="$(arg lidar_roll) $(arg lidar_pitch) $(arg lidar_yaw)" />
     <parent link="base_link"/>
     <child link="laser" />
@@ -38,9 +46,9 @@
           <box size="0.01 0.01 0.01" />
         </geometry>
-        <material name="grey" />
+        <material name="Grey" />
       </visual>
   </link>
   <joint name="base_link_to_laser_link2" type="fixed">
-    <origin xyz="-0.3955 0.0 0.211" rpy="0 0 ${PI}" />
+    <origin xyz="-0.390 0.0 0.211" rpy="0 0 ${PI}" />
     <parent link="base_link"/>
     <child link="laser_link2" />
@@ -52,5 +60,5 @@
           <box size="0.01 0.01 0.01" />
         </geometry>
-        <material name="grey" />
+        <material name="Grey" />
       </visual>
   </link>
@@ -66,9 +74,9 @@
           <box size="0.01 0.01 0.01" />
         </geometry>
-        <material name="grey" />
+        <material name="Grey" />
       </visual>
   </link>
   <joint name="camera" type="fixed">
-    <origin xyz="-0.38775 0.0 0.1807" rpy="1.5708 3.14159 4.71239"/>
+    <origin xyz="-0.384 0.0 0.1817" rpy="1.5708 3.14159 4.71239"/>
     <parent link="base_link"/>
     <child link="camera" />
@@ -80,5 +88,5 @@
           <box size="0.01 0.48 0.01" />
         </geometry>
-        <material name="transparentblack" />
+        <material name="TransparentBlack" />
       </visual>
   </link>
@@ -94,11 +102,32 @@
           <box size="0.01 0.01 0.01" />
         </geometry>
-        <material name="grey" />
+        <material name="Grey" />
       </visual>
   </link>
   <joint name="camera1_link" type="fixed">
-    <origin xyz="0.1749 0.0 0.0" rpy="0 0 0" />
+    <origin xyz="0.1553 0.0 0.0" rpy="0 0 0" />
     <parent link="base_link"/>
     <child link="camera1_link" />
   </joint>
+ <link name="base_Upperlink">
+   <visual>
+    <origin xyz=" 0 0 0 " rpy="0 0 0" />
+      <geometry>
+        <mesh
+          filename="package://tetra_description/meshes/ds4_m/platform_body_upper.stl" scale="0.001 0.001 0.001" />
+      </geometry>
+      <material name="TransparentRed"/>
+    </visual>
+      <collision>
+            <origin xyz="0 0 0" rpy="0 0 0"/>
+            <geometry>
+                <cylinder length="${base_length}" radius="${base_radius}"/>
+            </geometry>
+      </collision>
+  </link>
+  <joint name="base_Upperlink" type="fixed">
+    <origin xyz="0.0 0.0 0.0" rpy="0 0 0" />
+    <parent link="base_link"/>
+    <child link="base_Upperlink" />
+  </joint>
 </robot>
